Commit message: base map and project structure finished, need to chekc for collision attribute of urdf files importance

File: assets/line.urdf (robot description, URDF)
Before this commit: robot custom_line, 1 links, 0 joints
Links:
- link baseLink: geometry collision box size=1 0.2 0.01; visual box size=1 0.2 0.01

Commit message: made segments collisionless to avoid unwanted dynamics with the drones, removed unnecesary env prints, added comments for the rest to better understand current code

File: assets/line.urdf (robot description, URDF)
Before this commit: robot custom_line, 1 links, 0 joints
Links:
- link baseLink: geometry collision box size=0 0 0; visual box size=1 0.2 0.01
